File: pcb_designs/RC3/RC3.kicad_sch (KiCad schematic)
At the start: 46 parts, among them J1 Conn_01x07_Socket, J10 Comms & ADC, J11 I2C OLED, J12 Conn_01x04_Pin, J2 Conn_01x07_Socket, J3 DCC Out, J4 DC In, J5 Barrel_Jack_Switch, J6 GPIO, J7 I2C Off Board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

Commit message: PCB RC3 Update
PCB RC3 Layout Updated
Parts:
- removed D5, D6: WS2812B, LED_SMD:LED_WS2812B_PLCC4_5.0x5.0mm_P3.2mm, symbol LED:WS2812B
- added D5, D6: SK6812, LED_SMD:LED_SK6812_PLCC4_5.0x5.0mm_P3.2mm, symbol LED:SK6812
- J10: value Comms & ADC -> Comms/ADC
- J12: value Conn_01x04_Pin -> Test Points
- J3: value DCC Out -> TRACK
- J4: value DC In -> DC 12 - 16 V
- J7: value I2C Off Board -> I2C0
- JP1: value SolderJumper_2_Open -> Orientation
Connections:
- net +5V: now also D5.3 (VDD), D6.3 (VDD)
- net ADC1: now also J10.7 (Pin_7); no longer J10.8 (Pin_8)
- net ADC2: now also J10.5 (Pin_5); no longer J10.6 (Pin_6)
- net AGND: now also J10.6 (Pin_6); no longer J10.7 (Pin_7)
- net GNDPWR: now also D5.1 (VSS), D6.1 (VSS)
- net GPIO00: now also J10.3 (Pin_3); no longer J10.4 (Pin_4)
- net GPIO01: now also J10.4 (Pin_4); no longer J10.5 (Pin_5)
- net GPIO17: now also J10.8 (Pin_8); no longer J10.3 (Pin_3)
- net at J8.2 (Pin_2): now also D6.4 (DOUT)
- net at R13.2: now also D5.2 (DIN)
- new net: D5.4 (DOUT), D6.2 (DIN)
Other:
- note removed: "12V - 16V DC"
- note removed: "Test Points"
